Commit message: switch to gazebo_Fortress

File: src/livox_laser_simulation_RO2/urdf/mid360.xacro (robot description, xacro)
@@ -4,8 +4,11 @@
   <xacro:property name="laser_min_range" value="0.1"/>
   <xacro:property name="laser_max_range" value="200.0"/>
-  <xacro:property name="samples" value="70000"/>
   <xacro:property name="resolution" value="0.002"/>
   <xacro:property name="noise_mean" value="0.0"/>
   <xacro:property name="noise_stddev" value="0.01"/>
+  <xacro:property name="horizontal_samples" value="1024"/>
+  <xacro:property name="vertical_samples" value="64"/>
+  <xacro:property name="vertical_min_angle" value="${-7.22/180*M_PI}"/>
+  <xacro:property name="vertical_max_angle" value="${55.22/180*M_PI}"/>
   <xacro:property name="mass" value="0.4" />
   <xacro:property name="length" value="0.1" />
@@ -34,42 +37,36 @@
     </joint>
     <gazebo reference="${name}">
-      <sensor type="ray" name="${name}">
+      <sensor type="gpu_lidar" name="${name}">
         <pose>0 0 0 0 0 0</pose>
         <visualize>true</visualize>
         <update_rate>100</update_rate>
-        <!-- This ray plgin is only for visualization. -->
-        <plugin name="${name}_plugin" filename="libros2_livox.so">
-			<ray>
-			  <scan>
-				<horizontal>
-				<samples>10</samples>
-				<resolution>1</resolution>
-				<min_angle>${0}</min_angle>
-				<max_angle>${2*M_PI}</max_angle>
-				</horizontal>
-				<vertical>
-				<samples>360</samples>
-				<resolution>1</resolution>
-				<min_angle>${-7.22/180*M_PI}</min_angle>
-				<max_angle>${55.22/180*M_PI}</max_angle>
-				</vertical>
-			  </scan>
-			  <range>
-				<min>${laser_min_range}</min>
-				<max>${laser_max_range}</max>
-				<resolution>${resolution}</resolution>
-			  </range>
-			  <noise>
-				<type>gaussian</type>
-				<mean>${noise_mean}</mean>
-				<stddev>${noise_stddev}</stddev>
-			  </noise>
-			</ray>
-          <visualize>true</visualize>
-		  <samples>${samples}</samples>
-		  <downsample>1</downsample>
-		  <csv_file_name>$(find ros2_livox_simulation)/scan_mode/mid360.csv</csv_file_name>
-		  <topic>${topic}</topic>
-        </plugin>
+        <topic>${topic}</topic>
+        <always_on>true</always_on>
+        <lidar>
+          <scan>
+            <horizontal>
+              <samples>${horizontal_samples}</samples>
+              <resolution>1</resolution>
+              <min_angle>${-M_PI}</min_angle>
+              <max_angle>${M_PI}</max_angle>
+            </horizontal>
+            <vertical>
+              <samples>${vertical_samples}</samples>
+              <resolution>1</resolution>
+              <min_angle>${vertical_min_angle}</min_angle>
+              <max_angle>${vertical_max_angle}</max_angle>
+            </vertical>
+          </scan>
+          <range>
+            <min>${laser_min_range}</min>
+            <max>${laser_max_range}</max>
+            <resolution>${resolution}</resolution>
+          </range>
+          <noise>
+            <type>gaussian</type>
+            <mean>${noise_mean}</mean>
+            <stddev>${noise_stddev}</stddev>
+          </noise>
+        </lidar>
       </sensor>
     </gazebo>
